File: KiCad_project/powerSection.kicad_sch (KiCad schematic)
At the start: 61 parts, among them J10 Screw_Terminal_01x02, J11 Barrel_Jack_Switch, SW2 SW_SPDT_321, U10 TPS54202DDC, U7 fuse, U8 TPS5450DDAR, U9 TPS54202DDC

Commit message: update GND routing
Parts:
- added C10: 0.1uF, Capacitor_SMD:C_0603_1608Metric_Pad1.08x0.95mm_HandSolder, symbol symbol_library:C
Connections:
- net +3.3V: now also C10.1
- net GND: now also C10.2
Changed lines of the file:
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@@
+	)
+	(junction
+		(at 199.39 133.35)
+		(diameter 0)
+		(color 0 0 0 0)
 	)
 	(junction
@@
 	)
 	(junction
+		(at 199.39 144.78)
+		(diameter 0)
+		(color 0 0 0 0)
+	)
+	(junction
 		(at 146.05 170.18)
 		(diameter 0)
@@
 	(wire
 		(pts
+			(xy 212.09 133.35) (xy 212.09 135.89)
+		)
+		(stroke
+			(width 0)
+			(type default)
+		)
+	)
+	(wire
+		(pts
 			(xy 105.41 81.28) (xy 100.33 81.28)
 		)
@@
 	(wire
 		(pts
+			(xy 199.39 133.35) (xy 212.09 133.35)
+		)
+		(stroke
+			(width 0)
+			(type default)
+		)
+	)
+	(wire
+		(pts
 			(xy 55.88 36.83) (xy 67.31 36.83)
 		)
@@
 	(wire
 		(pts
+			(xy 199.39 144.78) (xy 212.09 144.78)
+		)
+		(stroke
+			(width 0)
+			(type default)
+		)
+	)
+	(wire
+		(pts
 			(xy 158.75 143.51) (xy 158.75 144.78)
 		)
@@
 		(pts
 			(xy 19.05 83.82) (xy 19.05 91.44)
+		)
+		(stroke
+			(width 0)
+			(type default)
+		)
+	)
+	(wire
+		(pts
+			(xy 212.09 143.51) (xy 212.09 144.78)
 		)
 		(stroke
@@
 					(unit 1)
 				)
+			)
+		)
+	)
+	(symbol
+		(lib_id "symbol_library:C")
+		(at 212.09 139.7 0)
+		(unit 1)
+		(exclude_from_sim no)
+		(in_bom yes)
+		(on_board yes)
+		(dnp no)
+		(property "Reference" "C10"
+			(at 215.9 138.4299 0)
+			(effects
+				(font
+					(size 1.27 1.27)
+				)
+				(justify left)
+			)
+		)
+		(property "Value" "0.1uF"
+			(at 216.154 140.716 0)
+			(effects
+				(font
+					(size 1.27 1.27)
+				)
+				(justify left)
+			)
+		)
+		(property "Footprint" "Capacitor_SMD:C_0603_1608Metric_Pad1.08x0.95mm_HandSolder"
+			(at 213.0552 143.51 0)
+			(effects
+				(font
+					(size 1.27 1.27)
+				)
+				(hide yes)
+			)
+		)
+		(property "Datasheet" "~"
+			(at 212.09 139.7 0)
+			(effects
+				(font
+					(size 1.27 1.27)
+				)
+				(hide yes)
+			)
+		)
+		(property "Description" "16V min"
+			(at 212.09 139.7 0)
+			(effects
+				(font
+					(size 1.27 1.27)
+				)
+				(hide yes)
+			)
+		)
+		(pin "1"
+		)
+		(pin "2"
+		)
+		(instances
+			(project "mobile_robot"
+				(path "/e8f9f0a0-cca9-426a-b8ab-73515fe7421d/7641e29b-8afb-4073-a9f3-cabc48dcae12"
+					(reference "C10")
+					(unit 1)
+				)
